File: GlowCoreMini.kicad_pcb (KiCad board)
At the start: 2 copper layers, 27.1 x 76.6 mm, 39 parts, among them J1 Conn_02x03_Counter_Clockwise, J2 DC-042C-Z-2.5-A, P1 WJ15EDGRC-3.81-3P, Q1 AP40P05, Q2 MMBT2222A, Q3 MMBT2222A, Q4 AP40P05, SW1 TS-1185EC-C-D-B, SW2 TS-1185EC-C-D-B, U1 SN74AHCT32QPWRQ1, U2 ESP32-WROOM-32E (4MB), U3 BL1117-33CX, U4 CP2102-GMR

Commit message: add warning info
Parts:
- removed D2: red LED, LED_SMD:LED_0603_1608Metric_Pad1.05x0.95mm_HandSolder
- removed J2: DC-042C-Z-2.5-A, DC-042C-Z-2:DC-IN-TH_DC-042C-Z-2.5-A
- removed MK1: ICS-43432, ICS-43432:MIC_ICS-43432
- removed Q1, Q4: AP40P05, Package_TO_SOT_SMD:SOT-23
- removed Q2, Q3: MMBT2222A, Package_TO_SOT_SMD:SOT-23
- removed R7: 1K, Resistor_SMD:R_0603_1608Metric_Pad0.98x0.95mm_HandSolder
- removed R8: 10K, Resistor_SMD:R_0603_1608Metric_Pad0.98x0.95mm_HandSolder
- removed REF**: OSHW-Logo2_7.3x6mm_SilkScreen, Symbol:OSHW-Logo2_7.3x6mm_SilkScreen
- added LED1: WS2812B-2020, footprint:LED-SMD_4P-L2.0-W2.0-TL_WS2812B-2020, F.Cu at (130.8, 94.1)
- added R4: 220, Resistor_SMD:R_0603_1608Metric_Pad0.98x0.95mm_HandSolder, F.Cu at (113.2, 124.3)
- added SW3: TS-1185EC-C-D-B, TS-1185EC-C-D-B:TS-1185EC-C-D-B, F.Cu at (124.1, 117.0)
- added U5: BL1117-33CX, Package_TO_SOT_SMD:SOT-223, F.Cu at (115.9, 119.0)
- added U6: UMH3N, footprint:SC-70-6_L2.2-W1.3-P0.65-LS2.1-BR, F.Cu at (127.7, 120.9)
- added U7: GMA4030H11-F26, GMA4030H11-F26:GMA4030H11-F26, F.Cu at (123.4, 121.2)
- C5: value 220uF 10V -> 10uF; footprint Capacitor_SMD:CP_Elec_6.3x5.4 -> Capacitor_SMD:C_0603_1608Metric_Pad1.08x0.95mm_HandSolder
- C8: value 10uF -> 1nF
- C9: value 1uF -> 1nF
- R2: value 100K -> 220
- U3: value BL1117-33CX -> KF350-3_5-2P; footprint Package_TO_SOT_SMD:SOT-223 -> footprint:CONN-TH_P3.50_KF350-3.5-2P
- moved C5 38.6 mm to (112.6, 112.7)
- moved U3 23.2 mm to (140.4, 142.8), turned to 0 degrees
- moved R5 11.7 mm to (129.7, 125.7)
- moved R6 11.4 mm to (130.1, 131.1)
Connections:
- C3 pad 2: +5V -> +3V3
- C4 pad 2: Net-(C4-Pad2) -> +5V
- C5 pad 1: +5V -> GND
- C5 pad 2: GND -> +3V3
- C8 pad 1: +3V3 -> RESET
- C9 pad 1: GND -> IO0
- C9 pad 2: RESET -> GND
- R2 pad 1: IO32/SD -> Net-(R2-Pad1)
- R2 pad 2: GND -> RESET
- R5 pad 1: RTS -> RESET
- R5 pad 2: Net-(Q2-Pad1) -> +3V3
- R6 pad 1: DTR -> IO0
- R6 pad 2: Net-(Q3-Pad1) -> +3V3
- SW1 pad 2: RESET -> Net-(R2-Pad1)
- SW2 pad 2: IO33/TESTBUTTON -> Net-(R4-Pad1)
- U3 pad 2: Net-(C4-Pad2) -> +5V
Routing:
- net GND: track 342.8 -> 0.00 mm, vias 11 -> 0
- net +5V: track 135.5 -> 0.00 mm, vias 11 -> 0
- net USB-C DATA-: track 88.8 -> 0.00 mm, vias 4 -> 0
- net LED1 DATA IN: track 86.4 -> 0.00 mm, vias 5 -> 0
- net +3V3: track 84.6 -> 0.00 mm, vias 3 -> 0
- net USB-C DATA+: track 83.9 -> 0.00 mm, vias 4 -> 0
- net RESET: track 80.7 -> 0.00 mm, vias 5 -> 0
- net IO13: track 45.1 -> 0.00 mm, vias 2 -> 0
- net IO33/TESTBUTTON: track 42.7 -> 0.00 mm, vias 2 -> 0
- net IO12: track 37.6 -> 0.00 mm, vias 1 -> 0
- net IO26/A0/DAC2: track 35.6 -> 0.00 mm, vias 1 -> 0
- net IO15/WS: track 34.1 -> 0.00 mm, vias 2 -> 0
- net RECEIVER 5V: track 33.7 -> 0.00 mm, vias 1 -> 0
- net IO25/A1/DAC1: track 31.9 -> 0.00 mm, vias 1 -> 0
- net IO14/SCK: track 27.7 -> 0.00 mm, vias 2 -> 0
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- removed copper zone on B.Cu, net GND
- removed copper zone on F.Cu, net GND
Other:
- board text added: "LED (IO13)"
- board text added: "dev board v1.0 beta 2"
- board text removed: "STATUS (IO13)"
- board text removed: "dev board v1.0 beta 1"
