File: GlowCoreMini PCB/GlowCoreMini PCB.kicad_sch (KiCad schematic)
At the start: 89 parts, among them P1 Solder_Pad, P10 Solder_Pad, P11 Solder_Pad, P12 Solder_Pad, P13 Solder_Pad, P14 Solder_Pad, P15 Solder_Pad, P16 Solder_Pad, P17 Solder_Pad, P18 Solder_Pad, P19 Solder_Pad, P2 Solder_Pad, P20 Solder_Pad, P21 Solder_Pad, P22 Solder_Pad, P3 Solder_Pad, P4 Solder_Pad, P5 Solder_Pad, P6 Solder_Pad, P7 Solder_Pad, P8 Solder_Pad, P9 Solder_Pad, SW1 TS24CA, SW2 TS24CA, SW3 TS24CA, U1 SN74LVC1G373DBVR, U10 LSM6DS3TR-C, U11 MSM261D4030H1CPM, U12 SPX3819M5-L-3-3_TR, U13 SK9822-EC20, U14 AP40P05, U15 AP40P05, U2 ESP32-S3-MINI-1-N8, U3 PTVSHC3N12VU, U4 AP40P05, U5 AP40P05, U6 AO3400A, U7 74LVC2G04DW-7, U8 AP40P05, U9 SN74LVC2T45DCUR

Commit message: updated pcb
Parts:
- JP1, JP2, P1, P10, P11, P12, P13, P14, P15, P16, P17, P18, P19, P2, P20, P21, P22, P3, P4, P5, P6, P7, P8, P9: now left out of the parts list
Changed lines of the file:
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@@
   )
   (symbol (lib_id "MyParts:Solder_Pad") (at 549.91 121.92 0) (unit 1)
-    (in_bom yes) (on_board yes) (dnp no) (fields_autoplaced)
+    (in_bom no) (on_board yes) (dnp no) (fields_autoplaced)
     (property "Reference" "P18" (at 558.8 120.6499 0)
       (effects (font (size 1.27 1.27)) (justify left))
@@
   )
   (symbol (lib_id "MyParts:Solder_Pad") (at 240.665 196.215 180) (unit 1)
-    (in_bom yes) (on_board yes) (dnp no) (fields_autoplaced)
+    (in_bom no) (on_board yes) (dnp no) (fields_autoplaced)
     (property "Reference" "P1" (at 236.855 188.595 0)
       (effects (font (size 1.27 1.27)))
@@
   )
   (symbol (lib_id "MyParts:Solder_Pad") (at 497.84 116.84 0) (unit 1)
-    (in_bom yes) (on_board yes) (dnp no) (fields_autoplaced)
+    (in_bom no) (on_board yes) (dnp no) (fields_autoplaced)
     (property "Reference" "P12" (at 506.73 115.5699 0)
       (effects (font (size 1.27 1.27)) (justify left))
@@
   )
   (symbol (lib_id "MyParts:Solder_Pad") (at 521.97 219.71 0) (unit 1)
-    (in_bom yes) (on_board yes) (dnp no) (fields_autoplaced)
+    (in_bom no) (on_board yes) (dnp no) (fields_autoplaced)
     (property "Reference" "P20" (at 530.86 218.4399 0)
       (effects (font (size 1.27 1.27)) (justify left))
@@
   )
   (symbol (lib_id "MyParts:Solder_Pad") (at 521.97 200.66 0) (unit 1)
-    (in_bom yes) (on_board yes) (dnp no) (fields_autoplaced)
+    (in_bom no) (on_board yes) (dnp no) (fields_autoplaced)
     (property "Reference" "P11" (at 530.86 199.3899 0)
       (effects (font (size 1.27 1.27)) (justify left))
@@
   )
   (symbol (lib_id "MyParts:Solder_Pad") (at 521.97 195.58 0) (unit 1)
-    (in_bom yes) (on_board yes) (dnp no) (fields_autoplaced)
+    (in_bom no) (on_board yes) (dnp no) (fields_autoplaced)
     (property "Reference" "P9" (at 530.86 194.3099 0)
       (effects (font (size 1.27 1.27)) (justify left))
@@
   )
   (symbol (lib_id "MyParts:Solder_Pad") (at 497.84 111.76 0) (unit 1)
-    (in_bom yes) (on_board yes) (dnp no) (fields_autoplaced)
+    (in_bom no) (on_board yes) (dnp no) (fields_autoplaced)
     (property "Reference" "P3" (at 506.73 110.4899 0)
       (effects (font (size 1.27 1.27)) (justify left))
@@
   )
   (symbol (lib_id "MyParts:Solder_Pad") (at 240.665 213.995 180) (unit 1)
-    (in_bom yes) (on_board yes) (dnp no) (fields_autoplaced)
+    (in_bom no) (on_board yes) (dnp no) (fields_autoplaced)
     (property "Reference" "P2" (at 236.855 206.375 0)
       (effects (font (size 1.27 1.27)))
@@
   )
   (symbol (lib_id "MyParts:Solder_Pad") (at 521.97 166.37 0) (unit 1)
-    (in_bom yes) (on_board yes) (dnp no) (fields_autoplaced)
+    (in_bom no) (on_board yes) (dnp no) (fields_autoplaced)
     (property "Reference" "P22" (at 530.86 165.0999 0)
       (effects (font (size 1.27 1.27)) (justify left))
@@
   )
   (symbol (lib_id "MyParts:Solder_Pad") (at 497.84 121.92 0) (unit 1)
-    (in_bom yes) (on_board yes) (dnp no) (fields_autoplaced)
+    (in_bom no) (on_board yes) (dnp no) (fields_autoplaced)
     (property "Reference" "P15" (at 506.73 120.6499 0)
       (effects (font (size 1.27 1.27)) (justify left))
@@
   )
   (symbol (lib_id "MyParts:Solder_Pad") (at 521.97 177.8 0) (unit 1)
-    (in_bom yes) (on_board yes) (dnp no) (fields_autoplaced)
+    (in_bom no) (on_board yes) (dnp no) (fields_autoplaced)
     (property "Reference" "P19" (at 530.86 176.5299 0)
       (effects (font (size 1.27 1.27)) (justify left))
@@
   )
   (symbol (lib_id "Jumper:SolderJumper_2_Open") (at 266.7 91.44 0) (unit 1)
-    (in_bom yes) (on_board yes) (dnp no) (fields_autoplaced)
+    (in_bom no) (on_board yes) (dnp no) (fields_autoplaced)
     (property "Reference" "JP1" (at 266.7 85.725 0)
       (effects (font (size 1.27 1.27)))
@@
   )
   (symbol (lib_id "MyParts:Solder_Pad") (at 549.91 111.76 0) (unit 1)
-    (in_bom yes) (on_board yes) (dnp no) (fields_autoplaced)
+    (in_bom no) (on_board yes) (dnp no) (fields_autoplaced)
     (property "Reference" "P16" (at 558.8 110.4899 0)
       (effects (font (size 1.27 1.27)) (justify left))
@@
   )
   (symbol (lib_id "MyParts:Solder_Pad") (at 521.97 184.15 0) (unit 1)
-    (in_bom yes) (on_board yes) (dnp no) (fields_autoplaced)
+    (in_bom no) (on_board yes) (dnp no) (fields_autoplaced)
     (property "Reference" "P7" (at 530.86 182.8799 0)
       (effects (font (size 1.27 1.27)) (justify left))
@@
   )
   (symbol (lib_id "MyParts:Solder_Pad") (at 521.97 172.72 0) (unit 1)
-    (in_bom yes) (on_board yes) (dnp no) (fields_autoplaced)
+    (in_bom no) (on_board yes) (dnp no) (fields_autoplaced)
     (property "Reference" "P6" (at 530.86 171.4499 0)
       (effects (font (size 1.27 1.27)) (justify left))
@@
   )
   (symbol (lib_id "MyParts:Solder_Pad") (at 521.97 207.01 0) (unit 1)
-    (in_bom yes) (on_board yes) (dnp no) (fields_autoplaced)
+    (in_bom no) (on_board yes) (dnp no) (fields_autoplaced)
     (property "Reference" "P14" (at 530.86 205.7399 0)
       (effects (font (size 1.27 1.27)) (justify left))
@@
   )
   (symbol (lib_id "MyParts:Solder_Pad") (at 521.97 189.23 0) (unit 1)
-    (in_bom yes) (on_board yes) (dnp no) (fields_autoplaced)
+    (in_bom no) (on_board yes) (dnp no) (fields_autoplaced)
     (property "Reference" "P8" (at 530.86 187.9599 0)
       (effects (font (size 1.27 1.27)) (justify left))
@@
   )
   (symbol (lib_id "MyParts:Solder_Pad") (at 521.97 224.79 0) (unit 1)
-    (in_bom yes) (on_board yes) (dnp no) (fields_autoplaced)
+    (in_bom no) (on_board yes) (dnp no) (fields_autoplaced)
     (property "Reference" "P10" (at 530.86 223.5199 0)
       (effects (font (size 1.27 1.27)) (justify left))
@@
   )
   (symbol (lib_id "MyParts:Solder_Pad") (at 521.97 161.29 0) (unit 1)
-    (in_bom yes) (on_board yes) (dnp no) (fields_autoplaced)
+    (in_bom no) (on_board yes) (dnp no) (fields_autoplaced)
     (property "Reference" "P21" (at 530.86 160.0199 0)
       (effects (font (size 1.27 1.27)) (justify left))
@@
   )
   (symbol (lib_id "MyParts:Solder_Pad") (at 549.91 116.84 0) (unit 1)
-    (in_bom yes) (on_board yes) (dnp no) (fields_autoplaced)
+    (in_bom no) (on_board yes) (dnp no) (fields_autoplaced)
     (property "Reference" "P17" (at 558.8 115.5699 0)
       (effects (font (size 1.27 1.27)) (justify left))
@@
   )
   (symbol (lib_id "MyParts:Solder_Pad") (at 521.97 212.09 0) (unit 1)
-    (in_bom yes) (on_board yes) (dnp no) (fields_autoplaced)
+    (in_bom no) (on_board yes) (dnp no) (fields_autoplaced)
     (property "Reference" "P13" (at 530.86 210.8199 0)
       (effects (font (size 1.27 1.27)) (justify left))
@@
   )
   (symbol (lib_id "Jumper:SolderJumper_2_Bridged") (at 328.93 290.195 0) (unit 1)
-    (in_bom yes) (on_board yes) (dnp no) (fields_autoplaced)
+    (in_bom no) (on_board yes) (dnp no) (fields_autoplaced)
     (property "Reference" "JP2" (at 328.93 283.845 0)
       (effects (font (size 1.27 1.27)))
@@
   )
   (symbol (lib_id "MyParts:Solder_Pad") (at 521.97 231.14 0) (unit 1)
-    (in_bom yes) (on_board yes) (dnp no) (fields_autoplaced)
+    (in_bom no) (on_board yes) (dnp no) (fields_autoplaced)
     (property "Reference" "P5" (at 530.86 229.8699 0)
       (effects (font (size 1.27 1.27)) (justify left))
@@
   )
   (symbol (lib_id "MyParts:Solder_Pad") (at 521.97 236.22 0) (unit 1)
-    (in_bom yes) (on_board yes) (dnp no) (fields_autoplaced)
+    (in_bom no) (on_board yes) (dnp no) (fields_autoplaced)
     (property "Reference" "P4" (at 530.86 234.9499 0)
       (effects (font (size 1.27 1.27)) (justify left))
